File: Hardware/KiCAD_Project_Files/Arduino_UNO_Shield_Template.sch (KiCad schematic (older format))
At the start: 5 parts, among them P1 HEADER_1X10, P2 HEADER_1X8, P3 HEADER_1X6, P4 HEADER_1X8, P5 HEADER_2X3

Commit message: Corrected ISP header net names in schematic Updated netlist connectivity in PCB Updated the pdf schematic
Connections:
- net labels removed: MISO, MOSI, SCK
Changed lines of the file:
@@
-EESchema Schematic File Version 2  date 1/31/2013 12:22:21 AM
+EESchema Schematic File Version 2  date 1/31/2013 1:20:18 AM
 LIBS:power
 LIBS:device
@@
 GND
 Text GLabel 5650 7200 0    40   Input ~ 0
-SCK
+IO13/SCK
 Text GLabel 5650 7100 0    40   Input ~ 0
-MISO
+IO12/MISO
 Text GLabel 6450 7200 2    40   Input ~ 0
-MOSI
+IO11/MOSI
 Text GLabel 5650 7300 0    40   Input ~ 0
 RESET

Commit message: Added notes & instructions to schematic and PCB file Added pdf of PCB drawing
Other:
- note added: "Use this schematic as a starting point and add components as needed. \nMake sure you keep existing reference designators when you annotate\nthe schematic. Otherwise the netlist will not line up with the board \nfile and the read netlist functionality will foobar the board design."
Changed lines of the file:
@@
-EESchema Schematic File Version 2  date 1/31/2013 1:20:18 AM
+EESchema Schematic File Version 2  date 2/12/2013 10:16:28 PM
 LIBS:power
 LIBS:device
@@
 Sheet 1 1
 Title ""
-Date "31 jan 2013"
+Date "13 feb 2013"
 Rev ""
 Comp ""
@@
 Comment4 ""
 $EndDescr
+Text Notes 3350 3050 0    100  ~ 0
+Use this schematic as a starting point and add components as needed.  \nMake sure you keep existing reference designators when you annotate\nthe schematic.  Otherwise the netlist will not line up with the board \nfile and the read netlist functionality will foobar the board design.
 $Comp
 L HEADER_2X3 P5
